File: KiCAD files/Effects_Pedals.kicad_pcb (KiCad board)
At the start: 2 copper layers, 226.1 x 53.1 mm, 155 parts, among them J1 OUT, J10 OUT, J11 Barrel_Jack_MountingPin, J2 IN, J3 IN, J4 OUT, J5 OUT, J6 IN, J7 IN, J8 OUT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

Commit message: Add new files
Parts:
- removed C39, C40, C42, C51: 0.1uF, Capacitor_THT:C_Disc_D3.0mm_W2.0mm_P2.50mm
- removed C48: 47pF, Capacitor_THT:C_Disc_D3.0mm_W2.0mm_P2.50mm
- removed C49: 0.01uF, Capacitor_THT:C_Disc_D3.0mm_W2.0mm_P2.50mm
- removed Compression: 25k, Connector_PinSocket_2.54mm:PinSocket_1x03_P2.54mm_Vertical
- removed D9: D, Diode_THT:D_DO-35_SOD27_P7.62mm_Horizontal
- removed Gain: 2k, Connector_PinSocket_2.54mm:PinSocket_1x03_P2.54mm_Vertical
- removed J5: OUT, Connector_PinHeader_1.00mm:PinHeader_1x02_P1.00mm_Vertical
- removed J6: IN, Connector_PinHeader_1.00mm:PinHeader_1x02_P1.00mm_Vertical
- removed Noise Gate: 500k, Connector_PinSocket_2.54mm:PinSocket_1x03_P2.54mm_Vertical
- removed PC41, PC45, PC47: 10uF, Capacitor_THT:CP_Radial_D4.0mm_P1.50mm
- removed PC43, PC46, PC50: 1uF, Capacitor_THT:CP_Radial_D4.0mm_P1.50mm
- removed PC44: 4.7uF, Capacitor_THT:CP_Radial_D4.0mm_P1.50mm
- removed Q2: NJFET, Package_TO_SOT_THT:TO-92_Inline
- removed R41, R45: 1k, Resistor_THT:R_Axial_DIN0207_L6.3mm_D2.5mm_P7.62mm_Horizontal
- removed R42: 100k, Resistor_THT:R_Axial_DIN0207_L6.3mm_D2.5mm_P7.62mm_Horizontal
- removed R43, R44, R46, R47: 10k, Resistor_THT:R_Axial_DIN0207_L6.3mm_D2.5mm_P7.62mm_Horizontal
- removed R48, R49, R50: 2.2M, Resistor_THT:R_Axial_DIN0207_L6.3mm_D2.5mm_P7.62mm_Horizontal
- removed the REF** at (48.5, 105.0)
- removed the REF** at (264.7, 61.6)
- removed the REF** at (48.5, 61.6)
- removed the REF** at (264.8, 105.0)
- removed Rotate: 50k, Connector_PinSocket_2.54mm:PinSocket_1x03_P2.54mm_Vertical
- removed U8: LM7805_TO220, Package_TO_SOT_THT:TO-220-3_Vertical
- removed U9: SSM2166, Package_SO:SO-14_3.9x8.65mm_P1.27mm
- added REF**: MountingHole_3.2mm_M3, MountingHole:MountingHole_3.2mm_M3, F.Cu at (221.5, 106.6)
- added REF**: MountingHole_3.2mm_M3, MountingHole:MountingHole_3.2mm_M3, F.Cu at (221.5, 61.9)
- added REF**: MountingHole_3.2mm_M3, MountingHole:MountingHole_3.2mm_M3, F.Cu at (44.2, 106.6)
- added REF**: MountingHole_3.2mm_M3, MountingHole:MountingHole_3.2mm_M3, F.Cu at (44.2, 61.9)
- moved J11 0.18 mm to (77.5, 65.0)
- moved C2 0.18 mm to (77.6, 68.7)
- moved C3 0.18 mm to (78.9, 72.7)
Routing:
- net Net-(U8-VO): track 71.5 -> 0.00 mm, vias 2 -> 0
- net PWR: track 50.4 -> 11.7 mm
- net Net-(U9-IN+): track 33.6 -> 0.00 mm, vias 2 -> 0
- net Net-(U9-ROT): track 32.3 -> 0.00 mm, vias 2 -> 0
- net Net-(U9-VCAGN): track 29.1 -> 0.00 mm, vias 1 -> 0
- net /Compressor/NG: track 28.4 -> 0.00 mm, vias 2 -> 0
- net Net-(U9-COMP): track 27.9 -> 0.00 mm, vias 4 -> 0
- net Net-(J5-Pin_1): track 19.7 -> 0.00 mm
- net Net-(Q2-S): track 16.7 -> 0.00 mm
- net Net-(U9-BUFOUT): track 16.5 -> 0.00 mm
- net Net-(U9-VCAIN): track 13.2 -> 0.00 mm, vias 2 -> 0
- net Net-(D9-K): track 12.9 -> 0.00 mm
- net Net-(U9-VCAR): track 12.7 -> 0.00 mm
- net Net-(C49-Pad2): track 11.3 -> 0.00 mm
- net Net-(U9-IN-): track 11.0 -> 0.00 mm
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- removed copper zone on F.Cu, net Net-(J6-Pin_1)
- removed copper zone on F.Cu, net Net-(Q2-G)
Other:
- board size 226.1 x 53.1 mm -> 188.2 x 55.5 mm
- board text added: "PT2399"
- board text removed: "COMPRESSOR"
