File: KiCAD files/Effects_Pedals.kicad_sch (KiCad schematic)
At the start: 0 parts

Commit message: Add new files
Other:
- removed sheet Compressor
Changed lines of the file:
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@@
 	)
 	(sheet
-		(at 34.29 106.68)
+		(at 106.68 106.68)
 		(size 50.8 38.1)
 		(exclude_from_sim no)
@@
 		)
 		(property "Sheetname" "Delay"
-			(at 34.29 105.9684 0)
+			(at 106.68 105.9684 0)
 			(effects
 				(font
@@
 		)
 		(property "Sheetfile" "Delay.kicad_sch"
-			(at 34.29 145.3646 0)
+			(at 106.68 145.3646 0)
 			(effects
 				(font
@@
 	)
 	(sheet
-		(at 100.33 106.68)
+		(at 172.72 106.68)
 		(size 63.5 39.37)
 		(exclude_from_sim no)
@@
 		)
 		(property "Sheetname" "Chorus"
-			(at 100.33 105.9684 0)
+			(at 172.72 105.9684 0)
 			(effects
 				(font
@@
 		)
 		(property "Sheetfile" "Chorus.kicad_sch"
-			(at 100.33 146.6346 0)
+			(at 172.72 146.6346 0)
 			(effects
 				(font
@@
 	)
 	(sheet
-		(at 177.8 106.68)
-		(size 78.74 40.64)
-		(exclude_from_sim no)
-		(in_bom yes)
-		(on_board yes)
-		(dnp no)
-		(fields_autoplaced yes)
-		(stroke
-			(width 0.1524)
-			(type solid)
-		)
-		(fill
-			(color 0 0 0 0.0000)
-		)
-		(property "Sheetname" "Compressor"
-			(at 177.8 105.9684 0)
-			(effects
-				(font
-					(size 1.27 1.27)
-				)
-				(justify left bottom)
-			)
-		)
-		(property "Sheetfile" "Compressor.kicad_sch"
-			(at 177.8 147.9046 0)
-			(effects
-				(font
-					(size 1.27 1.27)
-				)
-				(justify left top)
-			)
-		)
-		(instances
-			(project "Effects_Pedals"
-				(path "/e8c598df-7c41-4c1d-9f04-953345b4bea2"
-					(page "7")
-				)
-			)
-		)
-	)
-	(sheet
-		(at 58.42 52.07)
+		(at 64.77 52.07)
 		(size 67.31 41.91)
 		(exclude_from_sim no)
@@
 		)
 		(property "Sheetname" "OD_Dist"
-			(at 58.42 51.3584 0)
+			(at 64.77 51.3584 0)
 			(effects
 				(font
@@
 		)
 		(property "Sheetfile" "Drive.kicad_sch"
-			(at 58.42 94.5646 0)
+			(at 64.77 94.5646 0)
 			(effects
 				(font
